File: sfp_loopback.kicad_pcb (KiCad board)
At the start: 2 copper layers, 80 x 50 mm, 61 parts, among them J1 Conn_Coaxial, J101 SFP+, J2 USB_B_Micro, J3 Conn_01x02, J4 Conn_Coaxial, J5 RS_JMP, U1 74HC14, U101 LT1963AxQ-3.3, U102 ONET1191PRGT

Commit message: update to kicad9
Other:
- net class Default removed
- net class loop_trace removed
